File: docs/diagram/rv_dis_schematic.kicad_sch (KiCad schematic)
At the start: 9 parts

Commit message: push
Parts:
- renumbered even_lane0 to even_lane_i0, even_lane1 to even_lane_i1, odd_lane0 to odd_lane_i0, odd_lane1 to odd_lane_i1
Connections:
- net at odd_lane_i0. (alu_result[31:0]): now also forward_unit. (ev1_rs2_data[31:0])
- net at ID_EX_dispatch. (i1_opcode_ex[6:0]): now also register_file. (i1_rs2_data[31:0]); no longer odd_lane_i0. (alu_result[31:0])
- net at forward_unit. (ev1_rs2_data[31:0]): no longer odd_lane_i0. (alu_result[31:0])
- net at even_lane_i1. (alu_result[31:0]): now also forward_unit. (ev1_rs2_data[31:0])
- net at even_lane_i0. (alu_result[31:0]): now also forward_unit. (ev1_rs2_data[31:0])
- net at odd_lane_i1. (alu_result[31:0]): now also forward_unit. (ev1_rs2_data[31:0]); no longer ID_EX_dispatch. (i1_opcode_ex[6:0])
- net at register_file. (i1_rs2_data[31:0]): no longer ID_EX_dispatch. (i1_opcode_ex[6:0])
- net at decoder0. (rs2_use): now also register_file. (i1_rs2_data[31:0])
- net at decoder1. (rs2_use): now also register_file. (i1_rs2_data[31:0])
- new net: ID_EX_dispatch. (i1_opcode_ex[6:0]), odd_lane_i0. (alu_result[31:0])
- new net: forward_unit. (ev1_rs2_data[31:0]), odd_lane_i0. (alu_result[31:0])
- new net: even_lane_i1. (alu_result[31:0]), forward_unit. (ev1_rs2_data[31:0])
- new net: even_lane_i0. (alu_result[31:0]), forward_unit. (ev1_rs2_data[31:0])
- new net: ID_EX_dispatch. (i1_opcode_ex[6:0]), odd_lane_i1. (alu_result[31:0])
- new net: ID_EX_dispatch. (i1_opcode_ex[6:0]), forward_unit. (ev1_rs2_data[31:0]) (x14)
- new net: ID_EX_dispatch. (i1_opcode_ex[6:0]), register_file. (i1_rs2_data[31:0]) (x3)
- new net: decoder0. (rs2_use), register_file. (i1_rs2_data[31:0]) (x3)
- new net: decoder1. (rs2_use), register_file. (i1_rs2_data[31:0]) (x3)
- new net: forward_unit. (ev1_rs2_data[31:0]), odd_lane_i1. (alu_result[31:0])
- now unconnected: forward_unit. (ev1_rs2_data[31:0]), forward_unit. (ev1_rs2_data[31:0]), forward_unit. (ev1_rs2_data[31:0]), forward_unit. (ev1_rs2_data[31:0]), forward_unit. (ev1_rs2_data[31:0]), forward_unit. (ev1_rs2_data[31:0]), forward_unit. (ev1_rs2_data[31:0]), forward_unit. (ev1_rs2_data[31:0]), forward_unit. (ev1_rs2_data[31:0]), forward_unit. (ev1_rs2_data[31:0]), forward_unit. (ev1_rs2_data[31:0]), forward_unit. (ev1_rs2_data[31:0]), forward_unit. (ev1_rs2_data[31:0]), forward_unit. (ev1_rs2_data[31:0]), forward_unit. (ev1_rs2_data[31:0]), forward_unit. (ev1_rs2_data[31:0]), forward_unit. (ev1_rs2_data[31:0]), forward_unit. (ev1_rs2_data[31:0]), forward_unit. (ev1_rs2_data[31:0]), forward_unit. (ev1_rs2_data[31:0]), forward_unit. (ev1_rs2_data[31:0]), register_file. (i1_rs2_data[31:0]), register_file. (i1_rs2_data[31:0]), register_file. (i1_rs2_data[31:0]), register_file. (i1_rs2_data[31:0]), register_file. (i1_rs2_data[31:0]), register_file. (i1_rs2_data[31:0]), register_file. (i1_rs2_data[31:0]), register_file. (i1_rs2_data[31:0]), register_file. (i1_rs2_data[31:0]), register_file. (i1_rs2_data[31:0]), register_file. (i1_rs2_data[31:0])
Changed lines of the file:
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@@
 		(on_board yes)
 		(dnp no)
-		(property "Reference" "odd_lane0"
-			(at 193.04 72.39 0)
+		(property "Reference" "odd_lane_i0"
+			(at 193.548 72.39 0)
 			(do_not_autoplace yes)
 			(effects
@@
 			(project ""
 				(path "/f8bb78f3-53b1-48bb-976c-7ca56381b79f"
-					(reference "odd_lane0")
+					(reference "odd_lane_i0")
 					(unit 1)
 				)
@@
 		(on_board yes)
 		(dnp no)
-		(property "Reference" "even_lane1"
-			(at 193.294 114.3 0)
+		(property "Reference" "even_lane_i1"
+			(at 194.056 114.3 0)
 			(effects
 				(font
@@
 			(project ""
 				(path "/f8bb78f3-53b1-48bb-976c-7ca56381b79f"
-					(reference "even_lane1")
+					(reference "even_lane_i1")
 					(unit 1)
 				)
@@
 		(on_board yes)
 		(dnp no)
-		(property "Reference" "even_lane0"
-			(at 193.294 97.79 0)
+		(property "Reference" "even_lane_i0"
+			(at 194.056 97.79 0)
 			(effects
 				(font
@@
 			(project "rv_dis_schematic"
 				(path "/f8bb78f3-53b1-48bb-976c-7ca56381b79f"
-					(reference "even_lane0")
+					(reference "even_lane_i0")
 					(unit 1)
 				)
@@
 		(on_board yes)
 		(dnp no)
-		(property "Reference" "odd_lane1"
-			(at 193.04 51.054 0)
+		(property "Reference" "odd_lane_i1"
+			(at 193.548 50.8 0)
 			(do_not_autoplace yes)
 			(effects
@@
 			(project "rv_dis_schematic"
 				(path "/f8bb78f3-53b1-48bb-976c-7ca56381b79f"
-					(reference "odd_lane1")
+					(reference "odd_lane_i1")
 					(unit 1)
 				)

Commit message: push
Parts:
- removed decoder0, decoder1: ~, symbol RV-DIS:decoder
- removed even_lane_i0, even_lane_i1: ~, symbol RV-DIS:even_lane
- removed forward_unit: ~, symbol RV-DIS:forward_unit
- removed odd_lane_i0, odd_lane_i1: ~, symbol RV-DIS:odd_lane
- removed register_file: ~, symbol RV-DIS:register_file
Connections:
- now unconnected: ID_EX_dispatch. (i1_opcode_ex[6:0]), ID_EX_dispatch. (i1_opcode_ex[6:0]), ID_EX_dispatch. (i1_opcode_ex[6:0]), ID_EX_dispatch. (i1_opcode_ex[6:0]), ID_EX_dispatch. (i1_opcode_ex[6:0]), ID_EX_dispatch. (i1_opcode_ex[6:0]), ID_EX_dispatch. (i1_opcode_ex[6:0]), ID_EX_dispatch. (i1_opcode_ex[6:0]), ID_EX_dispatch. (i1_opcode_ex[6:0]), ID_EX_dispatch. (i1_opcode_ex[6:0]), ID_EX_dispatch. (i1_opcode_ex[6:0]), ID_EX_dispatch. (i1_opcode_ex[6:0]), ID_EX_dispatch. (i1_opcode_ex[6:0]), ID_EX_dispatch. (i1_opcode_ex[6:0]), ID_EX_dispatch. (i1_opcode_ex[6:0]), ID_EX_dispatch. (i1_opcode_ex[6:0]), ID_EX_dispatch. (i1_opcode_ex[6:0]), ID_EX_dispatch. (i1_opcode_ex[6:0]), ID_EX_dispatch. (i1_opcode_ex[6:0])
Other:
- added sheet s1_fetch (s1_fetch.kicad_sch)
- added sheet s2_decode (s2_decode.kicad_sch)
- added sheet s3_execute (s3_execute.kicad_sch)
- added sheet s4_memory (s4_memory.kicad_sch)
- added sheet s5_wback (s5_wback.kicad_sch)
- title: (none) -> RISC-V Dual-Issue SIMD Processor
