File: docs/diagram/rv_dis_schematic.kicad_sch (KiCad schematic)
At the start: 1 part

Commit message: push
Parts:
- removed ID_EX_dispatch: ~, symbol RV-DIS:ID_EX_dispatch
Other:
- sheet s3_execute renamed s4_execute
- sheet s4_memory renamed s5_memory
- removed sheet s5_wback
- added sheet s3_dispatch (s3_dispatch.kicad_sch)
- added sheet s6_wback (s6_wback.kicad_sch)
- sheet s4_execute: file s3_execute.kicad_sch -> s4_execute.kicad_sch
- sheet s5_memory: file s4_memory.kicad_sch -> s5_memory.kicad_sch

Commit message: push
Other:
- title: RISC-V Dual-Issue SIMD Processor -> RISC-V Dual-Issue Processor
Changed lines of the file:
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@@
 	(paper "A4")
 	(title_block
-		(title "RISC-V Dual-Issue SIMD Processor")
+		(title "RISC-V Dual-Issue Processor")
 		(date "2026-06-12")
 		(rev "v1.0")
