File: docs/diagram/s3_execute.kicad_sch (KiCad schematic)
At the start: 10 parts

Commit message: push
Parts:
- removed EX_MEM_even0, EX_MEM_even1: ~, symbol RV-DIS:EX_MEM_even
- removed EX_MEM_odd0, EX_MEM_odd1: ~, symbol RV-DIS:EX_MEM_odd
- removed ID_EX_dispatch: ~, symbol RV-DIS:ID_EX_dispatch
- removed even_lane_i0, even_lane_i1: ~, symbol RV-DIS:even_lane
- removed forward_unit: ~, symbol RV-DIS:forward_unit
- removed odd_lane0, odd_lane1: ~, symbol RV-DIS:odd_lane
Other:
- title: RISC-V Dual-Issue SIMD Processor -> (none)
