File: docs/diagram/s1_fetch.kicad_sch (KiCad schematic)
At the start: 0 parts

Commit message: push
Parts:
- added IF_ID: ~, symbol RV-DIS:IF_ID
- added instruction_cache: ~, symbol RV-DIS:instruction_cache
- added pc: ~, symbol RV-DIS:pc
- added pc_selector: ~, symbol RV-DIS:pc_selector
- added target_buffer: ~, symbol RV-DIS:target_buffer
Connections:
- new net: pc. (pc1_out[31:0]), pc_selector. (stall) (x3)
- new net: IF_ID. (i1_pc_target_id[31:0]), target_buffer. (i1_pc_target[31:0]) (x4)
- new net: IF_ID. (i1_pc_target_id[31:0]), instruction_cache. (i1_instr[31:0]) (x2)
- new net s3_dispatch: pc. (pc1_out[31:0])

Commit message: push
Connections:
- net at pc_selector. (stall): now also pc. (pc1_out[31:0])
- net at target_buffer. (i1_pc_target[31:0]): now also IF_ID. (i1_pc_target_id[31:0])
- net at IF_ID. (i1_pc_target_id[31:0]): no longer target_buffer. (i1_pc_target[31:0])
- net at instruction_cache. (i1_instr[31:0]): now also IF_ID. (i1_pc_target_id[31:0])
- new net: pc. (pc1_out[31:0]), pc_selector. (stall) (x2)
- new net: IF_ID. (i1_pc_target_id[31:0]), target_buffer. (i1_pc_target[31:0]) (x3)
- new net: IF_ID. (i1_pc_target_id[31:0]), instruction_cache. (i1_instr[31:0])
- now unconnected: IF_ID. (i1_pc_target_id[31:0]), IF_ID. (i1_pc_target_id[31:0]), IF_ID. (i1_pc_target_id[31:0]), IF_ID. (i1_pc_target_id[31:0]), IF_ID. (i1_pc_target_id[31:0])
Other:
- title: RISC-V Dual-Issue SIMD Processor -> RISC-V Dual-Issue Processor
Changed lines of the file:
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@@
 	(paper "A4")
 	(title_block
-		(title "RISC-V Dual-Issue SIMD Processor")
+		(title "RISC-V Dual-Issue Processor")
 		(date "2026-06-12")
 		(rev "v1.0")
