File: docs/diagram/s2_decode.kicad_sch (KiCad schematic)
At the start: 4 parts

Commit message: push
Parts:
- removed decoder1, decoder2: ~, symbol RV-DIS:decoder
- added Decoder_i0, Decoder_i1: ~, symbol RV-DIS:decoder
- added IF_ID: ~, symbol RV-DIS:IF_ID
- added state_buffer: ~, symbol RV-DIS:state_buffer
- added target_predict_i0, target_predict_i1: ~, symbol RV-DIS:target_predict
- renumbered ID_EX_dispatch to ID_DP
Connections:
- net at ID_DP. (ev1_imm_ex[31:0]): now also register_file1. (i1_rs1_data[31:0])
- net at register_file1. (i1_rs1_data[31:0]): no longer ID_DP. (ev1_imm_ex[31:0])
- new net: ID_DP. (ev1_imm_ex[31:0]), register_file1. (i1_rs1_data[31:0]) (x3)
- new net: Decoder_i0. (brch_en), state_buffer. (i1_target_state[1:0])
- new net: Decoder_i0. (brch_en), IF_ID. (i1_pc_target_id[31:0])
- new net: Decoder_i1. (brch_en), state_buffer. (i1_target_state[1:0])
- new net: Decoder_i1. (brch_en), IF_ID. (i1_pc_target_id[31:0])
- now unconnected: register_file1. (i1_rs1_data[31:0]), register_file1. (i1_rs1_data[31:0]), register_file1. (i1_rs1_data[31:0]), register_file1. (i1_rs1_data[31:0]), register_file1. (i1_rs1_data[31:0]), register_file1. (i1_rs1_data[31:0]), register_file1. (i1_rs1_data[31:0]), register_file1. (i1_rs1_data[31:0]), register_file1. (i1_rs1_data[31:0]), register_file1. (i1_rs1_data[31:0]), register_file1. (i1_rs1_data[31:0])
Other:
- moved on the sheet: register_file1

Commit message: push
Connections:
- net at ID_DP. (ev1_imm_ex[31:0]): now also register_file1. (i1_rs1_data[31:0])
- net at register_file1. (i1_rs1_data[31:0]): no longer ID_DP. (ev1_imm_ex[31:0])
- net at Decoder_i0. (brch_en): now also IF_ID. (i1_pc_target_id[31:0])
- net at state_buffer. (i1_target_state[1:0]): now also Decoder_i1. (brch_en); no longer Decoder_i0. (brch_en)
- net at IF_ID. (i1_pc_target_id[31:0]): no longer Decoder_i0. (brch_en)
- net at Decoder_i1. (brch_en): now also IF_ID. (i1_pc_target_id[31:0]); no longer state_buffer. (i1_target_state[1:0])
- new net: ID_DP. (ev1_imm_ex[31:0]), register_file1. (i1_rs1_data[31:0]) (x3)
- new net: Decoder_i0. (brch_en), state_buffer. (i1_target_state[1:0])
- now unconnected: IF_ID. (i1_pc_target_id[31:0]), register_file1. (i1_rs1_data[31:0]), register_file1. (i1_rs1_data[31:0]), register_file1. (i1_rs1_data[31:0])
Other:
- title: RISC-V Dual-Issue SIMD Processor -> RISC-V Dual-Issue Processor
Changed lines of the file:
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@@
 	(paper "A4")
 	(title_block
-		(title "RISC-V Dual-Issue SIMD Processor")
+		(title "RISC-V Dual-Issue Processor")
 		(date "2026-06-12")
 		(rev "v1.0")
