File: docs/diagram/s4_execute.kicad_sch (KiCad schematic)
At the start: 8 parts

Commit message: push
Connections:
- net at reserve_station_even. (ev1_rs2_data_fw): now also even_lane_i1. (alu_result[31:0])
- net at even_lane_i0. (alu_result[31:0]): no longer reserve_station_even. (ev1_rs2_data_fw)
- net at even_lane_i1. (alu_result[31:0]): no longer reserve_station_even. (ev1_rs2_data_fw)
- net at reserve_station_odd. (od0_rs2_data_fw): no longer DP_EX. (ev1_imm_ex[31:0])
- net at odd_lane_i1. (link_pc[31:0]): now also reserve_station_odd. (od0_rs2_data_fw)
- net at odd_lane_i0. (link_pc[31:0]): now also reserve_station_odd. (od0_rs2_data_fw)
- new net: DP_EX. (ev1_imm_ex[31:0]), reserve_station_even. (ev1_rs2_data_fw) (x12)
- new net: even_lane_i0. (alu_result[31:0]), reserve_station_even. (ev1_rs2_data_fw) (x2)
- new net: even_lane_i1. (alu_result[31:0]), reserve_station_even. (ev1_rs2_data_fw)
- new net: DP_EX. (ev1_imm_ex[31:0]), reserve_station_odd. (od0_rs2_data_fw) (x12)
- new net: odd_lane_i1. (link_pc[31:0]), reserve_station_odd. (od0_rs2_data_fw)
- new net: odd_lane_i0. (link_pc[31:0]), reserve_station_odd. (od0_rs2_data_fw)
- now unconnected: even_lane_i0. (alu_result[31:0]), even_lane_i1. (alu_result[31:0]), reserve_station_odd. (od0_rs2_data_fw), reserve_station_odd. (od0_rs2_data_fw), reserve_station_odd. (od0_rs2_data_fw), reserve_station_odd. (od0_rs2_data_fw), reserve_station_odd. (od0_rs2_data_fw), reserve_station_odd. (od0_rs2_data_fw), reserve_station_odd. (od0_rs2_data_fw), reserve_station_odd. (od0_rs2_data_fw), reserve_station_odd. (od0_rs2_data_fw), reserve_station_odd. (od0_rs2_data_fw), reserve_station_odd. (od0_rs2_data_fw), reserve_station_odd. (od0_rs2_data_fw), reserve_station_odd. (od0_rs2_data_fw), reserve_station_odd. (od0_rs2_data_fw), reserve_station_odd. (od0_rs2_data_fw)
Other:
- title: RISC-V Dual-Issue SIMD Processor -> RISC-V Dual-Issue Processor
Changed lines of the file:
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@@
 	(paper "A4")
 	(title_block
-		(title "RISC-V Dual-Issue SIMD Processor")
+		(title "RISC-V Dual-Issue Processor")
 		(date "2026-06-12")
 		(rev "v1.0")
