File: docs/diagram/s5_memory.kicad_sch (KiCad schematic)
At the start: 3 parts

Commit message: push
Connections:
- net at memory. (i1_mem_data[31:0]): now also EX_MEM_WB. (i0_wdata_wb[31:0])
- new net: EX_MEM_WB. (i0_wdata_wb[31:0]), memory. (i1_mem_data[31:0])
Other:
- title: RISC-V Dual-Issue SIMD Processor -> RISC-V Dual-Issue Processor
Changed lines of the file:
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@@
 	(paper "A4")
 	(title_block
-		(title "RISC-V Dual-Issue SIMD Processor")
+		(title "RISC-V Dual-Issue Processor")
 		(date "2026-06-12")
 		(rev "v1.0")
