File: docs/diagram/s6_wback.kicad_sch (KiCad schematic)
At the start: 1 part

Commit message: push
Other:
- title: RISC-V Dual-Issue SIMD Processor -> RISC-V Dual-Issue Processor
Changed lines of the file:
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@@
 	(paper "A4")
 	(title_block
-		(title "RISC-V Dual-Issue SIMD Processor")
+		(title "RISC-V Dual-Issue Processor")
 		(date "2026-06-12")
 		(rev "v1.0")
